Commit message: 카메라 위치 수정

File: desc/kobuki.urdf .xacro (robot description, xacro)
@@ -216,5 +216,5 @@
       <origin xyz="0 0 0" rpy="0 0 0"/>
       <geometry>
-        <box size="${cameraSize} ${cameraSize} ${cameraSize}"/>
+        <sphere radius= "0.02"/>
       </geometry>
     </collision>
@@ -222,5 +222,5 @@
       <origin xyz="0 0 0" rpy="0 0 0"/>
       <geometry>
-        <sphere radius= "0.03"/><!--"${cameraSize} ${cameraSize} ${cameraSize}"/>-->
+        <sphere radius= "0.02"/><!--"${cameraSize} ${cameraSize} ${cameraSize}"/>-->
       </geometry>
       <material name="green"/>
@@ -244,5 +244,5 @@
       <origin xyz="0 0 0" rpy="0 0 0"/>
       <geometry>
-        <box size="${cameraSize} ${cameraSize} ${cameraSize}"/>
+        <sphere radius= "0.02"/>
       </geometry>
     </collision>
@@ -250,5 +250,5 @@
       <origin xyz="0 0 0" rpy="0 0 0"/>
       <geometry>
-        <sphere radius= "0.03"/>
+        <sphere radius= "0.02"/>
       </geometry>
       <material name="green"/>
