Commit message: 눈알 두개 추가 최종

File: desc/kobuki.urdf.xacro (robot description, xacro)
@@ -212,5 +212,5 @@
     <xacro:property name="cameraSize" value="0.04"/>
     <xacro:property name="cameraMass" value="0.1"/>
-      <link name="my_right_camera">
+      <link name="my_left_camera">
     <collision>
       <origin xyz="0 0 0" rpy="0 0 0"/>
@@ -235,10 +235,10 @@
   <joint name="custom_camera_joint_right" type="fixed">
     <axis xyz="0 1 0" />
-    <origin xyz=".12 .11 .153" rpy="0 0 0"/>
+    <origin xyz=".12 .11 .153" rpy="0 0 0.6"/>
     <parent link="base_link"/>
-    <child link="my_right_camera"/>
+    <child link="my_left_camera"/>
   </joint>
   <!-- my_camera left-->
-       <link name="my_left_camera">
+       <link name="my_right_camera">
     <collision>
       <origin xyz="0 0 0" rpy="0 0 0"/>
@@ -263,7 +263,7 @@
   <joint name="custom_camera_joint_left" type="fixed">
     <axis xyz="0 1 0" />
-    <origin xyz=".12 -.11 .153" rpy="0 0 0"/>
+    <origin xyz=".12 -.11 .153" rpy="0 0 -0.6"/>
     <parent link="base_link"/>
-    <child link="my_left_camera"/>
+    <child link="my_right_camera"/>
   </joint>
     <!-- Kobuki Gazebo simulation details -->
