Commit message: Fix camera topic sub

File: desc/kobuki_gazebo.urdf.xacro (robot description, xacro)
@@ -178,5 +178,5 @@
     </gazebo>
     <gazebo reference="my_left_camera">
-      <material>Gazebo/Green</material>
+      <material>Gazebo/Black</material>
       <sensor type="camera" name="my_left_camera">
 	<update_rate>20.0</update_rate>
@@ -196,5 +196,5 @@
           <alwaysOn>true</alwaysOn>
           <updateRate>0.0</updateRate>
-          <cameraName>/my_right_camera/rgb</cameraName>
+          <cameraName>/my_left_camera/rgb</cameraName>
           <imageTopicName>image_raw</imageTopicName>
           <cameraInfoTopicName>camera_info</cameraInfoTopicName>
@@ -210,5 +210,5 @@
     </gazebo>
     <gazebo reference="my_right_camera">
-      <material>Gazebo/Green</material>
+      <material>Gazebo/Black</material>
       <sensor type="camera" name="my_right_camera">
 	<update_rate>20.0</update_rate>
